File: underwater2.sch (KiCad schematic (older format))
At the start: 78 parts, among them IC1 ICM-20948, J1 Motor1, J10 ICM20948 out, J11 Pow, J12 serial, J13 serial2, J14 5v pow, J15 5v pow, J2 Motor2, J3 Raspberry_Pi_2_3, J4 USB_C_Receptacle_USB2.0, J5 USB out, J6 Water, J7 Power, J8 Light, J9 MotorPow, SW1 SW_Push, U1 FT230XS, U2 TB6612FNG, U3 TB6612FNG, U4 ESP32-WROOM-32, U5 LM1117-1.8, U7 LM1117-3.3

Commit message: Modify milestone 2020724
Parts:
- removed C1: 10μF, Capacitor_SMD:C_1206_3216Metric, symbol Device:C_Small
- removed C14: 22μF10V, Capacitor_SMD:C_1206_3216Metric, symbol Device:C_Small
- removed C16: 2.2nF6.3V, Capacitor_SMD:C_1206_3216Metric, symbol Device:C_Small
- removed C2: 47pF, Capacitor_SMD:C_1206_3216Metric, symbol Device:C_Small
- removed C7: 4.7μF, Capacitor_SMD:C_1206_3216Metric, symbol Device:CP_Small
- removed D1: RX, Capacitor_SMD:C_1206_3216Metric, symbol Device:LED_Small
- removed D2: TX, Capacitor_SMD:C_1206_3216Metric, symbol Device:LED_Small
- removed J11: Pow, Connector_PinHeader_2.54mm:PinHeader_1x02_P2.54mm_Vertical, symbol Connector:Conn_01x02_Female
- removed J4: USB_C_Receptacle_USB2.0, DigiKey:USB-C_Female_E8124-015-01, symbol extend:USB_C_Receptacle_USB2.0_fixed
- removed J5: USB out, Connector_PinHeader_2.54mm:PinHeader_1x05_P2.54mm_Vertical, symbol Connector:Conn_01x05_Female
- removed JP1: High Full, Jumper:SolderJumper-3_P1.3mm_Open_RoundedPad1.0x1.5mm, symbol Jumper:SolderJumper_3_Open
- removed JP2: TX, Jumper:SolderJumper-2_P1.3mm_Open_Pad1.0x1.5mm, symbol Device:Jumper_NC_Small
- removed JP3: RX, Jumper:SolderJumper-2_P1.3mm_Open_Pad1.0x1.5mm, symbol Device:Jumper_NC_Small
- removed PS1: ACT4060ASH-T, SamacSys_Parts:SOIC127P605X175-8N, symbol SamacSys_Parts:ACT4060ASH-T
- removed R16: 1.5k Full, Capacitor_SMD:C_1206_3216Metric, symbol Device:R_Small
- removed R8: 10k, Capacitor_SMD:C_1206_3216Metric, symbol Device:R_Small
- removed SW1: SW_Push, Button_Switch_THT:SW_PUSH_6mm, symbol Switch:SW_Push
- removed U1: FT230XS, Package_SO:SSOP-16_3.9x4.9mm_P0.635mm, symbol Interface_USB:FT230XS
- added C10: 1nF/16V, Capacitor_SMD:C_0603_1608Metric, symbol Device:C_Small
- added C11: 22µF/10V, Capacitor_SMD:C_0603_1608Metric, symbol Device:C_Small
- added C5: 4.7μF, Capacitor_SMD:C_1206_3216Metric, symbol Device:C_Small
- added C6: 100nF, Capacitor_SMD:C_1206_3216Metric, symbol Device:C_Small
- added C7: 4.7nF/25V, Capacitor_SMD:C_0603_1608Metric, symbol Device:C_Small
- added C9: ifnecessary, Capacitor_SMD:C_1206_3216Metric, symbol Device:C_Small
- added D4: RX, Capacitor_SMD:C_1206_3216Metric, symbol Device:LED_Small
- added D6: POWER, Capacitor_SMD:C_1206_3216Metric, symbol Device:LED_Small
- added IC1, IC2: KST10MTF, SOT95P240X120-3N, symbol SamacSys_Parts:KST10MTF
- added IC3: ACT4070BYH-T, SOIC127P600X170-9N, symbol SamacSys_Parts:ACT4070BYH-T
- added J3: external regurator, Connector_PinSocket_2.54mm:PinSocket_1x03_P2.54mm_Vertical, symbol Connector:Conn_01x03_Female
- added J4: USB_C_Receptacle_USB2.0, DigiKey:USB-C_Female_E8124-015-01, symbol underwater2-rescue:USB_C_Receptacle_USB2.0_fixed-extend
- added J5: Pow, Connector_PinHeader_2.54mm:PinHeader_1x02_P2.54mm_Vertical, symbol Connector:Conn_01x02_Female
- added J8: Conn_01x10_Female, Connector_PinSocket_2.54mm:PinSocket_1x09_P2.54mm_Vertical, symbol Connector:Conn_01x09_Female
- added JP1: Jumper_NC_Small, Jumper:SolderJumper-2_P1.3mm_Open_RoundedPad1.0x1.5mm, symbol Device:Jumper_NC_Small
- added JP4: tx rx, symbol Device:Jumper_NC_Small
- added JP5: rx tx, symbol Device:Jumper_NC_Small
- added R11: 51k, Capacitor_SMD:C_0603_1608Metric, symbol Device:R_Small
- added R9: 270, Capacitor_SMD:C_1206_3216Metric, symbol Device:R_Small
- added SW1, SW2: SW_Push_Dual, Button_Switch_THT:SW_PUSH_6mm, symbol Switch:SW_Push_Dual
- added SW3: SW_DIP_x01, Button_Switch_THT:SW_E-Switch_EG1271_DPDT, symbol Switch:SW_DIP_x01
- added U1: FT232RL, Package_SO:SSOP-28_5.3x10.2mm_P0.65mm, symbol Interface_USB:FT232RL
- C1: renamed from C11; value 10nF50V -> 10nF/25V; footprint Capacitor_SMD:C_1206_3216Metric -> Capacitor_SMD:C_0603_1608Metric
- C2: renamed from C17; value 10μF35V -> 10µF/50V
- C3: value 47pF -> 10nF
- C8: value 100nF -> if necessary
- D3: value Power -> TX
- D5: renamed from D7; value 34/40V 3A -> 40V/3A
- FB1: value FB -> Ferrite_Bead_Small
- J11: renamed from J8; footprint Connector_PinHeader_2.54mm:PinHeader_1x03_P2.54mm_Horizontal -> Connector_PinHeader_2.54mm:PinHeader_1x03_P2.54mm_Vertical
- L1: value 15μH -> 15µH4A; footprint Capacitor_SMD:C_1206_3216Metric -> SamacSys_Parts:B952ASH100MP3
- R1, R2: value 5.1k -> 10k
- R10: value 10k -> 270
- R12: value 330k -> 9.76k; footprint Capacitor_SMD:C_1206_3216Metric -> Capacitor_SMD:C_0603_1608Metric
- R13: value 28.7k -> 330k
- R14: value 15k -> 12k; footprint Capacitor_SMD:C_1206_3216Metric -> Capacitor_SMD:C_0603_1608Metric
- R15: value 1.5k High -> 270
- R3: value 27 -> 10k
- R4: value 27 -> 5.1k
- R5: value 270 -> 5.1k
- R6, R7: value 270 -> 27
- renumbered C18 to C12, C19 to C13, C5 to C14, C9 to C15, C15 to C16, C12 to C17, C13 to C18, C6 to C19, C10 to C20, D5 to D1, D8 to D2, D6 to D7, D4 to D8, IC1 to IC4, J15 to J1, J7 to J10, J10 to J12, J1 to J14, J2 to J15, J9 to J16, J14 to J2, J3 to J6, J12 to J7, J6 to J9, JP4 to JP2, JP5 to JP3, R9 to R16, R11 to R8, U7 to U2, U2 to U3, U5 to U4, U4 to U5, U3 to U6
Connections:
- net labels added: +3.3V, +5V, ESP_EN, IO0
- wire segments 450 -> 521
- no-connect marks 58 -> 57
Other:
- moved on the sheet: C1, C12, C13, C14, C15, C16, C17, C18, C19, C2, C20, D1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

Commit message: Add broken charger.
Parts:
- removed J3: external regurator, Connector_PinSocket_2.54mm:PinSocket_1x03_P2.54mm_Vertical, symbol Connector:Conn_01x03_Female
- removed J5: Pow, Connector_PinHeader_2.54mm:PinHeader_1x02_P2.54mm_Vertical, symbol Connector:Conn_01x02_Female
- removed JP1: Jumper_NC_Small, Jumper:SolderJumper-2_P1.3mm_Open_RoundedPad1.0x1.5mm, symbol Device:Jumper_NC_Small
- added BT1: Battery, Connector_PinSocket_2.54mm:PinSocket_1x02_P2.54mm_Vertical, symbol Device:Battery
- added C21: 10μF, SamacSys_Parts:865080640004, symbol Device:CP_Small
- added C22, C23: 0.22μF, Capacitor_SMD:C_0603_1608Metric, symbol Device:C_Small
- added C24: 4.7uF, SamacSys_Parts:865080640004, symbol Device:CP_Small
- added C25: 10μF, Capacitor_SMD:C_0603_1608Metric, symbol Device:C_Small
- added C26: 0.1μF, Capacitor_SMD:C_0603_1608Metric, symbol Device:C_Small
- added D9: LED_Small, Capacitor_SMD:C_1206_3216Metric, symbol Device:LED_Small
- added IC5: MAX662ACSA+, SOIC127P600X175-8N, symbol SamacSys_Parts:MAX662ACSA+
- added IC6: MCP73842T-840I_UN, SOP50P490X110-10N, symbol SamacSys_Parts:MCP73842T-840I_UN
- added J10: momentary switch, Connector_PinHeader_2.54mm:PinHeader_1x04_P2.54mm_Vertical, symbol Connector:Conn_01x04_Female
- added J16: Conn_01x02_Female, Connector_PinHeader_2.54mm:PinHeader_1x02_P2.54mm_Vertical, symbol Connector:Conn_01x02_Female
- added J17, J18: Conn_01x02_Female, Connector_PinHeader_2.54mm:PinHeader_1x03_P2.54mm_Vertical, symbol Connector:Conn_01x03_Female
- added JP7: charge, Jumper:SolderJumper-2_P1.3mm_Open_RoundedPad1.0x1.5mm, symbol Device:Jumper_NO_Small
- added LED1, LED2, LED3, LED4, LED5, LED6: MP-2016-1100-65-70, MP201611006570, symbol SamacSys_Parts:MP-2016-1100-65-70
- added Q1, Q2, Q3, Q4, Q5, Q6, Q7, Q8: 2SC2712-Y,LF, SOT95P260X140-3N, symbol SamacSys_Parts:2SC2712-Y,LF
- added Q9: NDS8434, SOIC127P600X175-8N, symbol SamacSys_Parts:NDS8434
- added R12, R9: 1k, Capacitor_SMD:C_0603_1608Metric, symbol Device:R_Small
- added R13, R15, R16, R17, R18, R21: 67, Capacitor_SMD:C_0603_1608Metric, symbol Device:R_Small
- added R27: 100, Capacitor_SMD:C_0603_1608Metric, symbol Device:R_Small
- added R28: 100m, Capacitor_SMD:C_0603_1608Metric, symbol Device:R_Small
- added R29: 100k, Capacitor_SMD:C_0603_1608Metric, symbol Device:R_Small
- added R30: R_Variable, Capacitor_SMD:C_0603_1608Metric, symbol Device:R_Variable
- added R31: sermal1, Capacitor_SMD:C_1206_3216Metric, symbol Device:R_Small
- added R32: sermal2, Capacitor_SMD:C_1206_3216Metric, symbol Device:R_Small
- C1: renamed from C3; footprint Capacitor_SMD:C_1206_3216Metric -> Capacitor_SMD:C_0603_1608Metric
- C14, C16, C17, C18, C19, C6, FB1: footprint Capacitor_SMD:C_1206_3216Metric -> Capacitor_SMD:C_0603_1608Metric
- C15, C20: footprint Capacitor_SMD:C_1206_3216Metric -> SamacSys_Parts:865080640004
- C2: renamed from C4; footprint Capacitor_SMD:C_1206_3216Metric -> Capacitor_SMD:C_0603_1608Metric
- C3: renamed from C5; footprint Capacitor_SMD:C_1206_3216Metric -> Capacitor_SMD:C_0603_1608Metric
- C4: renamed from C8; footprint Capacitor_SMD:C_1206_3216Metric -> Capacitor_SMD:C_0603_1608Metric
- C5: renamed from C9; value ifnecessary -> if necessary; footprint Capacitor_SMD:C_1206_3216Metric -> Capacitor_SMD:C_0603_1608Metric
- C7: renamed from C12; footprint Capacitor_SMD:C_1206_3216Metric -> Capacitor_SMD:C_0603_1608Metric
- C8: renamed from C13; footprint Capacitor_SMD:C_1206_3216Metric -> Capacitor_SMD:C_0603_1608Metric
- D1, D8: footprint SamacSys_Parts:DIONM7959X282N -> SamacSys_Parts:DIOM5226X240N
- J11: value Light -> external regurator; footprint Connector_PinHeader_2.54mm:PinHeader_1x03_P2.54mm_Vertical -> Connector_PinSocket_2.54mm:PinSocket_1x03_P2.54mm_Vertical
- J5: renamed from J9; footprint Connector_PinHeader_2.54mm:PinHeader_1x02_P2.54mm_Horizontal -> Connector_PinHeader_2.54mm:PinHeader_1x02_P2.54mm_Vertical
- J9: renamed from J10; footprint Connector_PinHeader_2.54mm:PinHeader_1x02_P2.54mm_Horizontal -> Connector_PinHeader_2.54mm:PinHeader_1x03_P2.54mm_Vertical; symbol Connector:Conn_01x02_Female -> Connector:Conn_01x03_Female
- JP2: renamed from JP4; footprint (none) -> Jumper:SolderJumper-2_P1.3mm_Open_RoundedPad1.0x1.5mm
- JP3: renamed from JP5; footprint (none) -> Jumper:SolderJumper-2_P1.3mm_Open_RoundedPad1.0x1.5mm
- R1: renamed from R4; footprint Capacitor_SMD:C_1206_3216Metric -> Capacitor_SMD:C_0603_1608Metric
- R10: renamed from R3; footprint Capacitor_SMD:C_1206_3216Metric -> Capacitor_SMD:C_0603_1608Metric
- R11: renamed from R15; footprint Capacitor_SMD:C_1206_3216Metric -> Capacitor_SMD:C_0603_1608Metric
- R14: renamed from R16; footprint Capacitor_SMD:C_1206_3216Metric -> Capacitor_SMD:C_0603_1608Metric
- R19: renamed from R8; footprint Capacitor_SMD:C_1206_3216Metric -> Capacitor_SMD:C_0603_1608Metric
- R2: renamed from R5; footprint Capacitor_SMD:C_1206_3216Metric -> Capacitor_SMD:C_0603_1608Metric
- R23: renamed from R13; footprint Capacitor_SMD:C_1206_3216Metric -> Capacitor_SMD:C_0603_1608Metric
- R25: renamed from R17; footprint Capacitor_SMD:C_1206_3216Metric -> Capacitor_SMD:C_0603_1608Metric
- R26: renamed from R18; footprint Capacitor_SMD:C_1206_3216Metric -> Capacitor_SMD:C_0603_1608Metric
- R3: renamed from R6; footprint Capacitor_SMD:C_1206_3216Metric -> Capacitor_SMD:C_0603_1608Metric
- R4: renamed from R7; footprint Capacitor_SMD:C_1206_3216Metric -> Capacitor_SMD:C_0603_1608Metric
- R5: renamed from R1; footprint Capacitor_SMD:C_1206_3216Metric -> Capacitor_SMD:C_0603_1608Metric
- R6: renamed from R2; footprint Capacitor_SMD:C_1206_3216Metric -> Capacitor_SMD:C_0603_1608Metric
- R7: renamed from R9; footprint Capacitor_SMD:C_1206_3216Metric -> Capacitor_SMD:C_0603_1608Metric
- R8: renamed from R10; footprint Capacitor_SMD:C_1206_3216Metric -> Capacitor_SMD:C_0603_1608Metric
- renumbered C2 to C10, C7 to C11, C10 to C12, C11 to C13, C1 to C9, D3 to D2, D4 to D3, D6 to D4, D7 to D5, D2 to D6, D5 to D7, J8 to J1, J14 to J13, J16 to J14, J4 to J2, J6 to J3, J7 to J4, J13 to J6, J1 to J7, J2 to J8, JP2 to JP1, JP3 to JP4, JP6 to JP5, JP7 to JP6, R11 to R20, R12 to R22, R14 to R24, U5 to U4, U4 to U5
Connections:
- net +5V: now also J3.2 (5V), J3.4 (5V), J7.1 (Pin_1), J8.1 (Pin_1), J9.3 (Pin_3), U2.3 (VI), J10.4 (Pin_4), J16.1 (Pin_1), R12.2; no longer C2.1, C3.1, D1.1 (A), FB1.2, U1.20 (VCC), U1.4 (VCCIO)
- net -BATT: now also C1.2, C10.2, C13.2, C14.2, C15.2, C16.2, C17.2, C18.2, C19.1, C2.2, C20.2, C3.2, C4.2, C5.2, C6.2, C7.1, C8.1, D5.1 (K), D7.1 (A), IC3.4 (GND), IC4.18 (GND), IC4.20 (RESV_2), J11.2 (Pin_2), J12.2 (Pin_2), J14.2 (Pin_2), J2.A1 (GND), J2.A12 (GND), J2.B1 (GND), J2.B12 (GND), J2.SH (SHIELD), J3.14 (GND), J3.20 (GND), J3.25 (GND), J3.30 (GND), J3.34 (GND), J3.39 (GND), J3.6 (GND), J3.9 (GND), J7.2 (Pin_2), J8.2 (Pin_2), J9.1 (Pin_1), JP5.1 (A), JP6.2 (B), R1.1, R11.2, R2.1, R22.2, R23.2, R24.2, SW1.1, SW2.2, U1.18 (GND), U1.21 (GND), U1.25 (AGND), U1.7 (GND), U2.1 (GND), U3.10 (PGND2), U3.18 (GND), U3.3 (PGND1), U3.4 (PGND1), U3.9 (PGND2), U4.1 (GND), U4.15 (GND), U4.38 (GND), U4.39 (GND), U5.1 (GND), U6.10 (PGND2), U6.18 (GND), U6.3 (PGND1), U6.4 (PGND1), U6.9 (PGND2), BT1.2 (-), C21.2, C24.2, C25.2, C26.1, IC5.7 (GND), IC6.8 (VSS), J10.1 (Pin_1), J17.3 (Pin_3), J18.3 (Pin_3), Q3.2, Q4.2, Q5.2, Q6.2, Q7.2, Q8.2, R30.1, R32.2; no longer C14.1, C15.1, C19.2, C20.1, D8.2 (K), U3.13 (VM2), U3.14 (VM3), U3.24 (VM1), U6.13 (VM2), U6.14 (VM3), U6.24 (VM1)
- net ESP_EN: now also IC1.3 (COLLECTOR); no longer SW1.4
- net IO32: now reaches U3.15 (PWMB), U4.8 (IO32)
- net IO13: now reaches U3.16 (BIN2), U4.16 (IO13)
- net IO12: now reaches U3.17 (BIN1), U4.14 (IO12)
- net IO14: now reaches U3.19 (STBY), U4.13 (IO14)
- net IO27: now reaches U3.21 (AIN1), U4.12 (IO27)
- net IO26: now reaches U3.22 (AIN2), U4.11 (IO26)
- net IO25: now reaches U3.23 (PWMA), U4.10 (IO25)
- net IO33: now reaches U4.9 (IO33), U6.15 (PWMB)
- net IO4: now reaches U4.26 (IO4), U6.16 (BIN2)
- net IO16: now reaches U4.27 (IO16), U6.17 (BIN1)
- net IO17: now reaches U4.28 (IO17), U6.19 (STBY)
- net IO18: now reaches U4.30 (IO18), U6.21 (AIN1)
- net IO19: now reaches U4.31 (IO19), U6.22 (AIN2)
- net IO15: now reaches U4.23 (IO15), U6.23 (PWMA)
- net SDA: now reaches IC4.24 (SDA/SDI), J12.3 (Pin_3), R25.2, U4.33 (IO21)
- net SCL: now reaches IC4.23 (SCL/SCLK), J12.4 (Pin_4), R26.2, U4.36 (IO22)
- net at U4.29 (IO5): now also R27.1; no longer J11.2 (Pin_2)
- net TXD0: now reaches C8.2, J3.8 (GPIO14/TXD), J4.1 (Pin_1), J6.1 (Pin_1), JP3.2
- net TXD0: now also U4.35 (TXD0/IO1); no longer U4.34 (RXD0/IO3)
- net RXD0: now reaches C7.2, J3.10 (GPIO15/RXD), J4.2 (Pin_2), J6.2 (Pin_2), JP2.2
- net RXD0: now also U4.34 (RXD0/IO3); no longer U4.35 (TXD0/IO1)
- net power: now reaches U4.6 (IO34)
- net power: now also J9.2 (Pin_2); no longer J9.1 (Pin_1)
- net at J5.1 (Pin_1): now also R9.1; no longer U4.7 (IO35)
- net at C12.1, C13.1, JP4.2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: now also J11.1 (Pin_1)
- net at D1.2 (K), JP1.1: now also JP7.1
- net at C10.1, D6.2 (K), IC3.2 (IN)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: now also J11.3 (Pin_3)
- net +BATT: now reaches SW3.1
- net +BATT: now also C14.1, C15.1, C19.2, C20.1, D8.2 (K), U3.13 (VM2), U3.14 (VM3), U3.24 (VM1), U6.13 (VM2), U6.14 (VM3), U6.24 (VM1), BT1.1 (+), C25.1, IC6.9 (VBAT), J17.1 (Pin_1), J18.1 (Pin_1), Q9.5 (D_1), Q9.6 (D_2), Q9.7 (D_3), Q9.8 (D_4), R13.2, R15.2, R16.2, R17.2, R18.2, R21.2
- net USB_TXD: now reaches JP2.1, U1.1 (TXD)
- net USB_DCD: now reaches U1.10 (DCD)
- net USB_DCD: now also J1.4 (Pin_4); no longer J1.5 (Pin_5)
- net USBD+: now reaches R4.1, U1.15 (USBD+)
- net USBD-: now reaches R3.1, U1.16 (USBD-)
- net USB_NRESET: now reaches C6.1, D2.2 (A), D3.2 (A), D4.2 (A), J1.6 (Pin_6), U1.17 (3V3OUT), U1.19 (~RESET~)
- net USB_DTR: now reaches IC2.2 (EMITTER), J1.1 (Pin_1), R6.1, U1.2 (DTR)
- net USB_OSCI: now reaches J1.7 (Pin_7)
- net USB_OSCI: now also U1.27 (OSCI); no longer U1.26 (TEST)
- net USB_OSCO: now reaches J1.8 (Pin_8)
- net USB_OSCO: now also U1.28 (OSCO); no longer U1.27 (OSCI)
- net USB_TEST: now reaches J1.9 (Pin_9)
- net USB_TEST: now also U1.26 (TEST); no longer U1.28 (OSCO)
- net USB_RTS: now reaches IC1.2 (EMITTER), J1.2 (Pin_2), R10.1, U1.3 (RTS)
- net USB_RXD: now reaches JP3.1, U1.5 (RXD)
- net USB_RI: now reaches J1.3 (Pin_3), U1.6 (RI)
- net USB_DCR: now reaches U1.9 (DCR)
- net USB_DCR: now also J1.5 (Pin_5); no longer J1.4 (Pin_4)
- removed net GND: C1.2, C10.2, C13.2, C14.2, C15.2, C16.2, C17.2, C18.2, C19.1, C2.2, C20.2, C3.2, C4.2, C5.2, C6.2, C7.1, C8.1, D5.1 (K), D7.1 (A), IC3.4 (GND), IC4.18 (GND), IC4.20 (RESV_2), J11.3 (Pin_3), J12.2 (Pin_2), J14.2 (Pin_2), J2.A1 (GND), J2.A12 (GND), J2.B1 (GND), J2.B12 (GND), J2.SH (SHIELD), J3.14 (GND), J3.20 (GND), J3.25 (GND), J3.30 (GND), J3.34 (GND), J3.39 (GND), J3.6 (GND), J3.9 (GND), J5.2 (Pin_2), J7.2 (Pin_2), J8.2 (Pin_2), J9.2 (Pin_2), JP5.1 (A), JP6.2 (B), R1.1, R11.2, R2.1, R22.2, R23.2, R24.2, SW1.1, SW1.3, SW2.2, U1.18 (GND), U1.21 (GND), U1.25 (AGND), U1.7 (GND), U2.1 (GND), U3.10 (PGND2), U3.18 (GND), U3.3 (PGND1), U3.4 (PGND1), U3.9 (PGND2), U4.1 (GND), U4.15 (GND), U4.38 (GND), U4.39 (GND), U5.1 (GND), U6.10 (PGND2), U6.18 (GND), U6.3 (PGND1), U6.4 (PGND1), U6.9 (PGND2)
- new net: C2.1, C3.1, D1.1 (A), FB1.2, U1.20 (VCC), U1.4 (VCCIO)
- new net: IC6.1 (SENSE), Q9.1 (S_1), Q9.2 (S_2), Q9.3 (S_3), R28.1
- new net: IC6.10 (DRV), Q9.4 (G)
- new net: C21.1, D9.2 (A), IC5.6 (VOUT), IC6.2 (VDD), R28.2, R29.2
- new net: D9.1 (K), IC6.3 (STAT1)
- new net: IC6.4 (EN), R29.1
- new net: IC6.5 (THREF), R31.1
- new net: IC6.6 (THERM), R30.2, R31.2, R32.1
- new net: C26.2, IC6.7 (TIMER)
- new net: J5.2 (Pin_2), Q1.3, Q2.3, R12.1
- new net: C22.1, IC5.1 (C1-)
- new net: C22.2, IC5.2 (C1+)
- new net: C23.1, IC5.3 (C2-)
- new net: C23.2, IC5.4 (C2+)
- new net: LED1.1 (K_1), LED1.2 (K_2), Q3.3
- new net: LED1.3 (A_1), LED1.4 (A_2), R13.1
- new net: LED2.1 (K_1), LED2.2 (K_2), Q4.3
- new net: LED2.3 (A_1), LED2.4 (A_2), R15.1
- new net: LED3.1 (K_1), LED3.2 (K_2), Q5.3
- new net: LED3.3 (A_1), LED3.4 (A_2), R16.1
- new net: LED4.1 (K_1), LED4.2 (K_2), Q6.3
- new net: LED4.3 (A_1), LED4.4 (A_2), R17.1
- new net: LED5.1 (K_1), LED5.2 (K_2), Q7.3
- new net: LED5.3 (A_1), LED5.4 (A_2), R18.1
- new net: LED6.1 (K_1), LED6.2 (K_2), Q8.3
- new net: LED6.3 (A_1), LED6.4 (A_2), R21.1
- new net: Q1.1, Q2.2
- new net: Q2.1, R9.2
- new net +VSW: J10.2 (Pin_2), J10.3 (Pin_3), JP1.2, JP4.1
- new net LED_SW: J17.2 (Pin_2), J18.2 (Pin_2), Q3.1, Q4.1, Q5.1, Q6.1, Q7.1, Q8.1, R27.2
- new net VCC: C24.1, IC5.5 (VCC), JP7.2
- new net WATER: J16.2 (Pin_2), Q1.2, U4.7 (IO35)
- no-connect marks 57 -> 63
Other:
- note added: "Raspberry PI 3/4"
- note added: "USB-C\n"
- note added: "test 10K"
- moved on the sheet: C1, C10, C11, C12, C13, C14, C15, C16, C17, C18, C19, C2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

Commit message: Modified drive ESC and external switch.
Parts:
- removed C14, C19, C26: 0.1μF, Capacitor_SMD:C_0603_1608Metric, symbol Device:C_Small
- removed C15, C20, C21: 10μF, SamacSys_Parts:865080640004, symbol Device:CP_Small
- removed C22, C23: 0.22μF, Capacitor_SMD:C_0603_1608Metric, symbol Device:C_Small
- removed C24: 4.7uF, SamacSys_Parts:865080640004, symbol Device:CP_Small
- removed C25: 10μF, Capacitor_SMD:C_0603_1608Metric, symbol Device:C_Small
- removed D8: DIODE, SamacSys_Parts:DIOM5226X240N, symbol Simulation_SPICE:DIODE
- removed D9: LED_Small, Capacitor_SMD:C_1206_3216Metric, symbol Device:LED_Small
- removed IC5: MAX662ACSA+, SOIC127P600X175-8N, symbol SamacSys_Parts:MAX662ACSA+
- removed IC6: MCP73842T-840I_UN, SOP50P490X110-10N, symbol SamacSys_Parts:MCP73842T-840I_UN
- removed J13: Motor1, Connector_PinSocket_2.54mm:PinSocket_1x04_P2.54mm_Horizontal, symbol Connector:Conn_01x04_Female
- removed J14: MotorPow, Connector_PinHeader_2.54mm:PinHeader_1x02_P2.54mm_Vertical, symbol Connector:Conn_01x02_Female
- removed J15: Motor2, Connector_PinSocket_2.54mm:PinSocket_1x04_P2.54mm_Horizontal, symbol Connector:Conn_01x04_Female
- removed J9: Power, Connector_PinHeader_2.54mm:PinHeader_1x03_P2.54mm_Vertical, symbol Connector:Conn_01x03_Female
- removed Q9: NDS8434, SOIC127P600X175-8N, symbol SamacSys_Parts:NDS8434
- removed R30: R_Variable, Capacitor_SMD:C_0603_1608Metric, symbol Device:R_Variable
- removed U3, U6: TB6612FNG, Package_SO:SSOP-24_5.3x8.2mm_P0.65mm, symbol Driver_Motor:TB6612FNG
- added D10, D11, D12, D9: 34/40V 3A, SamacSys_Parts:DIOM5226X240N, symbol Simulation_SPICE:DIODE
- added D8: Pwr 5V, Capacitor_SMD:C_1206_3216Metric, symbol Device:LED_Small
- added F1: fuse 10A, Resistor_SMD:R_1206_3216Metric, symbol Device:Fuse_Small
- added IC5: KST10MTF, SOT95P240X120-3N, symbol SamacSys_Parts:KST10MTF
- added J13: Water Sence, Connector_PinHeader_2.54mm:PinHeader_1x02_P2.54mm_Vertical, symbol Connector:Conn_01x02_Female
- added J14: LED Left, Connector_PinHeader_2.54mm:PinHeader_1x03_P2.54mm_Vertical, symbol Connector:Conn_01x03_Female
- added J15: LED right, Connector_PinHeader_2.54mm:PinHeader_1x03_P2.54mm_Vertical, symbol Connector:Conn_01x03_Female
- added J19: BLMOTOR_B2, Connector_PinHeader_2.54mm:PinHeader_1x03_P2.54mm_Vertical, symbol Connector:Conn_01x03_Female
- added J20: BLMOTOR_B1, Connector_PinHeader_2.54mm:PinHeader_1x03_P2.54mm_Vertical, symbol Connector:Conn_01x03_Female
- added J21: BLMOTOR_A2, Connector_PinHeader_2.54mm:PinHeader_1x03_P2.54mm_Vertical, symbol Connector:Conn_01x03_Female
- added J22: BLMOTOR_A1, Connector_PinHeader_2.54mm:PinHeader_1x03_P2.54mm_Vertical, symbol Connector:Conn_01x03_Female
- added J23: BATT Chrg, Connector_PinSocket_2.54mm:PinSocket_1x02_P2.54mm_Vertical, symbol Connector:Conn_01x02_Female
- added J24, J25: BT pow, Connector_PinHeader_2.54mm:PinHeader_1x02_P2.54mm_Vertical, symbol Connector:Conn_01x02_Female
- added J9: PJ1-021-SMT-TR, PJ1021SMTTR, symbol SamacSys_Parts:PJ1-021-SMT-TR
- added JP8: SolderJumper_3_Open, Jumper:SolderJumper-3_P1.3mm_Open_RoundedPad1.0x1.5mm, symbol Jumper:SolderJumper_3_Open
- added Q10: IRLML6344TRPBF, SOT95P237X112-3N, symbol SamacSys_Parts:IRLML6344TRPBF
- added Q9: DMP3099L-7, SOT96P240X120-3N, symbol SamacSys_Parts:DMP3099L-7
- added R30: 39k, Capacitor_SMD:C_0603_1608Metric, symbol Device:R_Small
- added R33, R34, R35, R36: 100, Capacitor_SMD:C_0603_1608Metric, symbol Device:R_Small
- BT1: value Battery -> BATT in
- D4: value POWER -> Pwr USB
- D5: value Power 3.3 -> Pwr 3.3V
- D6: footprint SamacSys_Parts:DIONM7959X282N -> SamacSys_Parts:DIOM5226X240N
- J1: value Conn_01x10_Female -> test con
- J11: value external regurator -> ext regurator
- J16: value Conn_01x02_Female -> Water con
- J17: value Conn_01x02_Female -> LED left con
- J18: value Conn_01x02_Female -> LED right con
- JP4: value J battpower -> BATT power
- R28: value 100m -> 270
- R31: value sermal1 -> 1k; footprint Capacitor_SMD:C_1206_3216Metric -> Capacitor_SMD:C_0603_1608Metric
- R32: value sermal2 -> 100k; footprint Capacitor_SMD:C_1206_3216Metric -> Capacitor_SMD:C_0603_1608Metric
Connections:
- net VCC is gone; now on net +5V: JP7.2
- net +3V3: now also J16.1 (Pin_1), J17.1 (Pin_1), J18.1 (Pin_1), R12.2, R13.2, R15.2, R16.2, R17.2, R18.2, R21.2, JP8.3 (B)
- net +5V: now also J10.1 (Pin_1), R28.1, JP8.1 (A), Q9.3; no longer J10.4 (Pin_4), J16.1 (Pin_1), R12.2
- net +BATT: now also D6.1 (A), SW3.2, D10.1 (A), D11.1 (A), D12.1 (A), D9.1 (A), J24.1 (Pin_1), J25.1 (Pin_1); no longer BT1.1 (+), J17.1 (Pin_1), J18.1 (Pin_1), R13.2, R15.2, R16.2, R17.2, R18.2, R21.2, SW3.1
- net +VSW: now also J10.4 (Pin_4), R29.2, Q9.2; no longer J10.2 (Pin_2), J10.3 (Pin_3)
- net -BATT: now also J10.2 (Pin_2), D8.1 (K), IC5.2 (EMITTER), J14.3 (Pin_3), J15.3 (Pin_3), J19.3 (Pin_3), J20.3 (Pin_3), J21.3 (Pin_3), J22.3 (Pin_3), J23.2 (Pin_2), J24.2 (Pin_2), J25.2 (Pin_2), J9.2, J9.3, Q10.2; no longer J10.1 (Pin_1)
- net IO15: now also R33.1
- net IO25: now also R35.1
- net IO32: now also R36.1
- net IO33: now also R34.1
- net LED_SW: now also J14.2 (Pin_2), J15.2 (Pin_2)
- net WATER: now also J13.2 (Pin_2)
- net GPIO5: now reaches J3.29 (GCLK1/GPIO5)
- net GPIO5: now also R30.2
- net GPIO6: now reaches J3.31 (GCLK2/GPIO6)
- net GPIO6: now also R31.2
- net at R28.2: now also D8.2 (A); no longer R29.2
- net at R29.1: now also IC5.3 (COLLECTOR), Q10.3, Q9.1
- net at R31.1: now also IC5.1 (BASE)
- net at R32.1: now also J10.3 (Pin_3), Q10.1, R30.1; no longer R31.2
- new net: BT1.1 (+), F1.1
- new net: J13.1 (Pin_1), J14.1 (Pin_1), J15.1 (Pin_1), JP8.2 (C)
- new net: J23.1 (Pin_1), J9.1
- new net: F1.2, SW3.1
- new net: D12.2 (K), J22.1 (Pin_1)
- new net: J22.2 (Pin_2), R36.2
- new net: D11.2 (K), J21.1 (Pin_1)
- new net: J21.2 (Pin_2), R35.2
- new net: D10.2 (K), J20.1 (Pin_1)
- new net: J20.2 (Pin_2), R34.2
- new net: D9.2 (K), J19.1 (Pin_1)
- new net: J19.2 (Pin_2), R33.2
- no-connect marks 63 -> 60
Other:
- note removed: "test 10K"
- moved on the sheet: BT1, C1, C10, C11, C12, C13, C16, C17, C18, C2, C3, C4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
